File: Canary.sch (KiCad schematic (older format))
At the start: 48 parts

Commit message: Clean up, add notes
Other:
- note added: "Run Iq: 0.6uA typ, 1uA max"
- note added: "Shutdown Iq: 0.3uA typ, 0.6uA max\nRun: 430uA typ, 900uA max"
- note added: "Shutdown Iq: 0.3uA typ, 1.2uA max\nRun: 3.3mA typ"
- note added: "Shutdown Iq: 0.6uA typ, 8uA max\nRun: 10uA typ, 18uA max"
- note added: "Shutdown Iq: 1uA typ, 10uA max\nRun: 5mA typ, 20mA max"
- note added: "Shutdown Iq: 34uA typ, 105uA max\nRun: 2.6mA typ, 3mA max"
- note added: "Shutdown Iq: 6uA max\nRun Iq: 130uA typ, 200uA max"
- note added: "Shutdown Iq: ~5mA\nRun: 60mA typ, 100mA max"
- note removed: "Shutdown Iq: 0.3uA typ, 0.6uA max"
- note removed: "Shutdown Iq: 0.6uA typ, 8uA max"
- note removed: "Shutdown Iq: 1uA typ, 10uA max"
- note removed: "Shutdown Iq: 34uA typ, 105uA max"
- note removed: "Shutdown Iq: 6uA max"
- moved on the sheet: C?, U?
Changed lines of the file:
@@
 L Device:C C?
 U 1 1 60A91FEF
-P 7750 3700
-F 0 "C?" H 7865 3746 50  0000 L CNN
-F 1 "0.1u" H 7865 3655 50  0000 L CNN
-F 2 "" H 7788 3550 50  0001 C CNN
-F 3 "~" H 7750 3700 50  0001 C CNN
-	1    7750 3700
+P 7750 3750
+F 0 "C?" H 7865 3796 50  0000 L CNN
+F 1 "0.1u" H 7865 3705 50  0000 L CNN
+F 2 "" H 7788 3600 50  0001 C CNN
+F 3 "~" H 7750 3750 50  0001 C CNN
+	1    7750 3750
 	-1   0    0    -1
 $EndComp
@@
 L JetkovKiCADLib:SHTC3 U?
 U 1 1 603451FE
-P 8200 3700
-F 0 "U?" H 8000 4050 50  0000 C CNN
-F 1 "SHTC3" H 8350 4050 50  0000 C CNN
-F 2 "JetkovKiCADLib:MCP7383xx-xxxx_OT" H 7700 3050 50  0001 L BNN
-F 3 "https://media.digikey.com/pdf/Data%20Sheets/Sensirion%20PDFs/HT_DS_SHTC3_D1.pdf" H 8450 3600 50  0001 L BNN
-F 4 "SHTC3" H 8250 3200 40  0001 C CNN "Part Number"
-F 5 "Sensirion AG" H 8250 3200 40  0001 C CNN "Manufacturer"
-F 6 "SENSOR HUMI/TEMP I2C 2% SMD" H 8250 3200 40  0001 C CNN "Description"
-F 7 "-40°C +125°C" H 8250 3200 40  0001 C CNN "Temp Range"
-	1    8200 3700
+P 8200 3750
+F 0 "U?" H 8000 4100 50  0000 C CNN
+F 1 "SHTC3" H 8350 4100 50  0000 C CNN
+F 2 "JetkovKiCADLib:MCP7383xx-xxxx_OT" H 7700 3100 50  0001 L BNN
+F 3 "https://media.digikey.com/pdf/Data%20Sheets/Sensirion%20PDFs/HT_DS_SHTC3_D1.pdf" H 8450 3650 50  0001 L BNN
+F 4 "SHTC3" H 8250 3250 40  0001 C CNN "Part Number"
+F 5 "Sensirion AG" H 8250 3250 40  0001 C CNN "Manufacturer"
+F 6 "SENSOR HUMI/TEMP I2C 2% SMD" H 8250 3250 40  0001 C CNN "Description"
+F 7 "-40°C +125°C" H 8250 3250 40  0001 C CNN "Temp Range"
+	1    8200 3750
 	1    0    0    -1
 $EndComp
 Text Notes 7850 1450 0    79   ~ 0
 VOC Sensor
-Text Notes 7850 3100 0    79   ~ 0
+Text Notes 7850 3150 0    79   ~ 0
 Humidity + \nTemperature\nSensor
 Text Notes 7950 2500 0    40   ~ 0
@@
 	1    0    0    -1
 $EndComp
-Text Notes 7950 4100 0    40   ~ 0
+Text Notes 7950 4150 0    40   ~ 0
 Address: 0x70\nFreq: 0 to 1MHz
 Wire Wire Line
-	8650 3800 8650 3850
+	8650 3850 8650 3900
 $Comp
 L power:GND #PWR?
 U 1 1 60AC8A96
-P 8650 3850
-F 0 "#PWR?" H 8650 3600 50  0001 C CNN
-F 1 "GND" H 8655 3677 50  0000 C CNN
-F 2 "" H 8650 3850 50  0001 C CNN
-F 3 "" H 8650 3850 50  0001 C CNN
-	1    8650 3850
-	-1   0    0    -1
-$EndComp
-Wire Wire Line
-	7750 3500 7750 3550
-Connection ~ 7750 3500
+P 8650 3900
+F 0 "#PWR?" H 8650 3650 50  0001 C CNN
+F 1 "GND" H 8655 3727 50  0000 C CNN
+F 2 "" H 8650 3900 50  0001 C CNN
+F 3 "" H 8650 3900 50  0001 C CNN
+	1    8650 3900
+	-1   0    0    -1
+$EndComp
+Wire Wire Line
+	7750 3550 7750 3600
+Connection ~ 7750 3550
 $Comp
 L power:GND #PWR?
 U 1 1 60A91FF5
-P 7750 3850
-F 0 "#PWR?" H 7750 3600 50  0001 C CNN
-F 1 "GND" H 7755 3677 50  0000 C CNN
-F 2 "" H 7750 3850 50  0001 C CNN
-F 3 "" H 7750 3850 50  0001 C CNN
-	1    7750 3850
-	-1   0    0    -1
-$EndComp
-Text GLabel 8650 3600 2    50   Input ~ 0
+P 7750 3900
+F 0 "#PWR?" H 7750 3650 50  0001 C CNN
+F 1 "GND" H 7755 3727 50  0000 C CNN
+F 2 "" H 7750 3900 50  0001 C CNN
+F 3 "" H 7750 3900 50  0001 C CNN
+	1    7750 3900
+	-1   0    0    -1
+$EndComp
+Text GLabel 8650 3650 2    50   Input ~ 0
 I2C_SCL
-Text GLabel 8650 3500 2    50   BiDi ~ 0
+Text GLabel 8650 3550 2    50   BiDi ~ 0
 I2C_SDA
 Text GLabel 8650 1950 2    50   Input ~ 0
@@
 $EndComp
 Wire Wire Line
-	7750 3450 7750 3500
+	7750 3500 7750 3550
 $Comp
 L power:VDD #PWR?
 U 1 1 60AB3D1B
-P 7750 3450
-F 0 "#PWR?" H 7750 3300 50  0001 C CNN
-F 1 "VDD" H 7765 3623 50  0000 C CNN
-F 2 "" H 7750 3450 50  0001 C CNN
-F 3 "" H 7750 3450 50  0001 C CNN
-	1    7750 3450
+P 7750 3500
+F 0 "#PWR?" H 7750 3350 50  0001 C CNN
+F 1 "VDD" H 7765 3673 50  0000 C CNN
+F 2 "" H 7750 3500 50  0001 C CNN
+F 3 "" H 7750 3500 50  0001 C CNN
+	1    7750 3500
 	1    0    0    -1
 $EndComp
@@
 Text GLabel 4300 2000 2    50   Input ~ 0
 CHG_STAT
-Text Notes 7750 4200 0    40   ~ 0
-Shutdown Iq: 0.3uA typ, 0.6uA max
-Text Notes 7800 2600 0    40   ~ 0
-Shutdown Iq: 34uA typ, 105uA max
-Text Notes 13600 2400 0    40   ~ 0
-Shutdown Iq: 6uA max
-Text Notes 13550 5100 0    40   ~ 0
-Shutdown Iq: 0.6uA typ, 8uA max
-Text Notes 2950 5250 0    40   ~ 0
-Shutdown Iq: 1uA typ, 10uA max
+Text Notes 7800 2700 0    40   ~ 0
+Shutdown Iq: 34uA typ, 105uA max\nRun: 2.6mA typ, 3mA max
+Text Notes 13550 2400 0    40   ~ 0
+Shutdown Iq: 6uA max\nRun Iq: 130uA typ, 200uA max
+Text Notes 13550 5150 0    40   ~ 0
+Shutdown Iq: 0.6uA typ, 8uA max\nRun: 10uA typ, 18uA max
+Text Notes 2950 5300 0    40   ~ 0
+Shutdown Iq: 1uA typ, 10uA max\nRun: 5mA typ, 20mA max
 $Comp
 L power:+3V3 #PWR?
@@
 	-1   0    0    -1
 $EndComp
+Text Notes 7400 5900 0    40   ~ 0
+Shutdown Iq: ~5mA\nRun: 60mA typ, 100mA max
+Text Notes 13550 6900 0    40   ~ 0
+Run Iq: 0.6uA typ, 1uA max
+Text Notes 7750 4350 0    40   ~ 0
+Shutdown Iq: 0.3uA typ, 0.6uA max\nRun: 430uA typ, 900uA max
+Text Notes 2750 3800 0    40   ~ 0
+Shutdown Iq: 0.3uA typ, 1.2uA max\nRun: 3.3mA typ
 $EndSCHEMATC

Commit message: Cleanup
Parts:
- removed C? (x2): DNP, symbol Device:C
- removed C?: 1u, symbol Device:C
- removed C? (x4): 0.1u, symbol Device:C
- removed R?: 49R9, symbol Device:R
- removed R?: 499k, symbol Device:R
- removed R?: 1M, symbol Device:R
- removed R? (x2): DNP, symbol Device:R
- removed U?: SPEC-110-902, JetkovKiCADLib:MIC2288YD5, symbol JetkovKiCADLib:SPEC-110-902
- removed U?: LMP91000, JetkovKiCADLib:LMP91000, symbol JetkovKiCADLib:LMP91000
- removed U?: MCP6041T-I_OT, JetkovKiCADLib:MCP6041T-I_OT, symbol JetkovKiCADLib:MCP6041T-I_OT
- removed U?: MAX6071BAUT21T, JetkovKiCADLib:MAX6071BAUT21, symbol JetkovKiCADLib:MAX6071BAUT21T
- C?: value 0.1u -> DNP
Connections:
- net 3V3_PS: now also J?.41 (P0.23)
- net 5V_EN: now also J?.6 (P0.25)
- net CHG_STAT: now also J?.40 (P0.22)
- net LED_AMBER: now also J?.10 (P0.29)
- net LED_GREEN: now also J?.11 (P0.30)
- net LED_RED: now also J?.9 (P0.28)
- net LMP_VOUT_B: now also J?.21 (P0.05/AIN3)
- net PIEZO_PWM: now also J?.12 (P0.31)
- net PM_UART_RXD: now also J?.25 (P0.09/NFC1)
- net PM_UART_TXD: now also J?.26 (P0.10/NFC2)
- net SPI_CLK: now also J?.32 (P0.14/TRACEDATA[3])
- net SPI_MISO: now also J?.34 (P0.16/TRACEDATA[1])
- net SPI_MOSI: now also J?.33 (P0.15/TRACEDATA[2])
- net SWDCLK: now also J?.44 (SWDIO)
- net SWDIO: now also J?.43 (SWCLK)
- net SWO: now also J?.36 (P0.18/TRACEDATA[0]/SWO)
- net VDD_EN: now also J?.42 (P0.24)
- net VREF_EN: now also J?.7 (P0.26)
- net ~FLASH_CS~: now also J?.35 (P0.17)
- net ~LMP_EN~: now also J?.8 (P0.27)
- net ~PM_SLEEP~: now also J?.27 (P0.11)
- net ~RESET~: now also J?.39 (P0.21/~RESET)
- net at J?.19 (P0.03/AIN1): now also R?.1, R?.2
Other:
- note added: "6 months sleep: 6*30*24h * (30e-3)mA = 130mAh\n3 days run: 3*24h * 10mA = 720mAh\n\nTotal: 850mAh\nEst. True Total: 500mAh"
- note added: "Humidity + Temperature Sensor"
- note added: "MCU + BLE"
- note added: "PM Sensor Connector"
- note added: "Power Consumption Rough Max Estimates"
- note added: "SWD Connector"
- note added: "Sensors"
- note added: "Sleep Total Iq: \n(2+1+7+1.2+10)uA/85% + 5uA = 30uA max\n\nSensor/Comm Duty Cycle:\n15s/(10*60s) = 2.5%\n\nRun Total:\n3.3V: [3.3mA + (2.5%)(2.6+5+0.5+0.5)mA]/85% = 5mA max\n5.0V: (2.5%)(100+0.5)mA/85% = 3mA max -> 5mA @ 3.3V"
- note added: "TODO\n- Jellybean BOM\n- Review"
- note added: "nRF52832"
- note removed: "2.048V Reference"
- note removed: "Address: 0x48\nFreq: 10 to 100kHz"
- note removed: "Humidity + \nTemperature\nSensor"
- note removed: "PM Sensor"
- note removed: "Potentiostat AFE"
- note removed: "Potentiostat\nOutput Buffer"
- note removed: "Run Iq: 0.6uA typ, 1uA max"
- note removed: "Shutdown Iq: 0.6uA typ, 8uA max\nRun: 10uA typ, 18uA max"
- note removed: "Shutdown Iq: 6uA max\nRun Iq: 130uA typ, 200uA max"
- note removed: "TODO\n- Passives for potentiostat\n- SPI flash\n- Connect everything to MCU\n- Calculate sleep mode power\n- Jellybean BOM"
- moved on the sheet: C?, D?, J?, LS?, Q?, R?, U?, Y?

Commit message: Select caps
Parts:
- added C?: 0.1u, JetkovKiCADLib:C_0402_NoSilk, symbol Device:C
- C? (x2): value C -> 12pF; footprint (none) -> JetkovKiCADLib:C_0402_NoSilk; Description (none) -> CAP CER 12PF 50V C0G/NP0 0402; Manufacturer (none) -> Samsung Electro-Mechanics; Part Number (none) -> CL05C120JB5NNNC; Temp Range (none) -> -55°C +125°C
- C? (x3): footprint (none) -> JetkovKiCADLib:C_0402_NoSilk; Description (none) -> CAP CER 1UF 10V X5R 0402; Manufacturer (none) -> Samsung Electro-Mechanics; Part Number (none) -> CL05A105KP5NNNC; Temp Range (none) -> -55°C +85°C
- C? (x3): footprint (none) -> JetkovKiCADLib:C_0402_NoSilk; Description (none) -> CAP CER 0.1UF 10V X5R 0402; Manufacturer (none) -> Samsung Electro-Mechanics; Part Number (none) -> CL05A104KP5NNNC; Temp Range (none) -> -55°C +85°C
- R? (x8): footprint (none) -> JetkovKiCADLib:R_0402_NoSilk
- R?: value ? -> 2.4M; footprint (none) -> JetkovKiCADLib:R_0402_NoSilk
- R?: value ? -> 2M; footprint (none) -> JetkovKiCADLib:R_0402_NoSilk
Connections:
- net +BATT: now also R?.2; no longer R?.1
- net GND: now also C?.2
- net XTAL1: now reaches C?.1, J?.13 (P0.00/XTAL1), Y?.2
- net XTAL2: now reaches C?.2, J?.14 (P0.01/XTAL2), Y?.1
- net BAT_DIV: now reaches J?.20 (P0.04/AIN2)
- net BAT_DIV: now also R?.1, R?.1, C?.1
- net PDRIVE_O: now reaches LS?.1, Q?.1 (D), Q?.1 (D), Q?.2 (D), Q?.2 (D), Q?.5 (D), Q?.5 (D), Q?.6 (D), Q?.6 (D)
- net PDRIVE: now reaches Q?.1 (D), Q?.2 (D), Q?.5 (D), Q?.6 (D), R?.1, R?.1, R?.2
- now unconnected: J?.19 (P0.03/AIN1)
Other:
- note added: "4.4V -> 2.4V\n"
- note added: "C1 = C2 = 2(C_L - C_stray)\nC1 = C2 = 2(9-3) = 12pF"
- moved on the sheet: C?, R?

Commit message: Add pizeo
Parts:
- removed LS?: Speaker_Crystal, symbol Device:Speaker_Crystal
- added LS?: PKMCS0909E4000-R1, JetkovKiCADLib:PKMCS0909E4000-R1, symbol JetkovKiCADLib:PKMCS0909E4000-R1
Changed lines of the file:
@@
 	4500 3550 4500 3600
-$Comp
-L Device:Speaker_Crystal LS?
-U 1 1 605E7267
-P 3200 6700
-F 0 "LS?" H 3100 6800 50  0000 L CNN
-F 1 "Speaker_Crystal" H 3375 6605 50  0001 L CNN
-F 2 "" H 3165 6650 50  0001 C CNN
-F 3 "~" H 3165 6650 50  0001 C CNN
-	1    3200 6700
-	1    0    0    -1
-$EndComp
 $Comp
 L power:+5V #PWR0134
@@
 Text Label 1650 6700 0    40   ~ 0
 PDRIVE
+$Comp
+L JetkovKiCADLib:PKMCS0909E4000-R1 LS?
+U 1 1 603826A5
+P 3200 6700
+F 0 "LS?" H 3100 6850 50  0000 L CNN
+F 1 "PKMCS0909E4000-R1" H 3100 6350 50  0000 L CNN
+F 2 "JetkovKiCADLib:PKMCS0909E4000-R1" H 3215 6350 50  0001 C CNN
+F 3 "https://www.murata.com/~/media/webrenewal/products/sound/sounder/vppt-buzj083-d.ashx" H 3165 6650 50  0001 C CNN
+F 4 "PKMCS0909E4000-R1" H 3150 6400 40  0001 C CNN "Part Number"
+F 5 "Murata Electronics" H 3150 6400 40  0001 C CNN "Manufacturer"
+F 6 "AUDIO PIEZO TRANSDUCER 12.5V SMD" H 3250 6400 40  0001 C CNN "Description"
+F 7 "-40°C +85°C" H 3150 6400 40  0001 C CNN "Temp Range"
+	1    3200 6700
+	1    0    0    -1
+$EndComp
 $EndSCHEMATC

Commit message: Fix part info, start rough layout
Parts:
- U2: renamed from U?; footprint JetkovKiCADLib:MCP7383xx-xxxx_OT -> JetkovKiCADLib:SHTC3
- U3: renamed from U?; footprint JetkovKiCADLib:MCP7383xx-xxxx_OT -> JetkovKiCADLib:SGP40-D-R4
- gave numbers to parts that had none: 31
Other:
- note added: "TODO\n- Jellybean BOM\n- Review\n- Button"
- note removed: "TODO\n- Jellybean BOM\n- Review"

Commit message: Adjust layour
Parts:
- added S?: SM-UART-04L, JetkovKiCADLib:SM-UART-04L, symbol JetkovKiCADLib:SM-UART-04L
- added SW1: TL3301SPF160QG, JetkovKiCADLib:TL3301SPF160QG, symbol JetkovKiCADLib:TL3301SPF160QG
Other:
- note added: "6 months sleep: 6*30*24h * (30e-3)mA = 130mAh\n3 days run: 3*24h * 10mA = 720mAh\n\nMax Total: 850mAh\nEst. Realistic Total: 500mAh"
- note removed: "6 months sleep: 6*30*24h * (30e-3)mA = 130mAh\n3 days run: 3*24h * 10mA = 720mAh\n\nTotal: 850mAh\nEst. True Total: 500mAh"
Changed lines of the file:
@@
 Power Consumption Rough Max Estimates
 Text Notes 8100 6150 0    59   ~ 0
-6 months sleep: 6*30*24h * (30e-3)mA = 130mAh\n3 days run: 3*24h * 10mA = 720mAh\n\nTotal: 850mAh\nEst. True Total: 500mAh
+6 months sleep: 6*30*24h * (30e-3)mA = 130mAh\n3 days run: 3*24h * 10mA = 720mAh\n\nMax Total: 850mAh\nEst. Realistic Total: 500mAh
 Wire Notes Line
 	6150 7500 750  7500
@@
 	1    0    0    -1
 $EndComp
+$Comp
+L JetkovKiCADLib:TL3301SPF160QG SW1
+U 1 1 603B5FDC
+P 12200 4550
+F 0 "SW1" H 12200 4835 50  0000 C CNN
+F 1 "TL3301SPF160QG" H 12200 4744 50  0000 C CNN
+F 2 "JetkovKiCADLib:TL3301SPF160QG" H 12100 4750 50  0001 C CNN
+F 3 "https://sten-eswitch-13110800-production.s3.amazonaws.com/system/asset/product_line/data_sheet/158/TL3301.pdf" H 12100 4750 50  0001 C CNN
+F 4 "TL3301SPF160QG" H 12200 4550 40  0001 C CNN "Part Number"
+F 5 "E-Switch" H 12200 4550 40  0001 C CNN "Manufacturer"
+F 6 "SWITCH TACTILE SPST-NO 0.05A 12V" H 12200 4550 40  0001 C CNN "Description"
+F 7 "-20°C +70°C" H 12200 4550 40  0001 C CNN "Temp Range"
+	1    12200 4550
+	1    0    0    -1
+$EndComp
+$Comp
+L JetkovKiCADLib:SM-UART-04L S?
+U 1 1 603C9AA9
+P 12000 5150
+F 0 "S?" H 12078 5188 40  0000 L CNN
+F 1 "SM-UART-04L" H 12078 5112 40  0000 L CNN
+F 2 "JetkovKiCADLib:SM-UART-04L" H 12000 4950 40  0001 C CNN
+F 3 "https://www.amphenol-sensors.com/en/component/edocman/514-telaire-sm-uart-04l-laser-dust-sensor-application-note/download?Itemid=8488%20%27" H 12000 5150 40  0001 C CNN
+F 4 "SM-UART-04L" H 12000 4950 40  0001 C CNN "Part Number"
+F 5 "Amphenol Advanced Sensors" H 12000 4950 40  0001 C CNN "Manufacturer"
+F 6 "PM2.5 IR LASER DUST SENSOR" H 12000 4950 40  0001 C CNN "Description"
+F 7 "-10°C +50°C" H 12000 4950 40  0001 C CNN "Temp Range"
+	1    12000 5150
+	1    0    0    -1
+$EndComp

Commit message: Update switch, placement adjustments
Parts:
- added H1: MountingHole, Mounting_Holes:MountingHole_2.2mm_M2, symbol Mechanical:MountingHole
- SW1: value TL3301SPF160QG -> TL3301SPF160QJ; footprint JetkovKiCADLib:TL3301SPF160QG -> JetkovKiCADLib:TL3301EF160QJ; Part Number TL3301SPF160QG -> TL3301SPF160QJ
- gave numbers to parts that had none: 1
Changed lines of the file:
@@
 L JetkovKiCADLib:TL3301SPF160QG SW1
 U 1 1 603B5FDC
-P 12200 4550
-F 0 "SW1" H 12200 4835 50  0000 C CNN
-F 1 "TL3301SPF160QG" H 12200 4744 50  0000 C CNN
-F 2 "JetkovKiCADLib:TL3301SPF160QG" H 12100 4750 50  0001 C CNN
-F 3 "https://sten-eswitch-13110800-production.s3.amazonaws.com/system/asset/product_line/data_sheet/158/TL3301.pdf" H 12100 4750 50  0001 C CNN
-F 4 "TL3301SPF160QG" H 12200 4550 40  0001 C CNN "Part Number"
-F 5 "E-Switch" H 12200 4550 40  0001 C CNN "Manufacturer"
-F 6 "SWITCH TACTILE SPST-NO 0.05A 12V" H 12200 4550 40  0001 C CNN "Description"
-F 7 "-20°C +70°C" H 12200 4550 40  0001 C CNN "Temp Range"
-	1    12200 4550
+P 12150 4600
+F 0 "SW1" H 12150 4885 50  0000 C CNN
+F 1 "TL3301SPF160QJ" H 12150 4794 50  0000 C CNN
+F 2 "JetkovKiCADLib:TL3301EF160QJ" H 12050 4800 50  0001 C CNN
+F 3 "https://www.digikey.ca/htmldatasheets/production/2066007/0/0/1/TL3301SPF160QJ-Drawing.pdf" H 12050 4800 50  0001 C CNN
+F 4 "TL3301SPF160QJ" H 12150 4600 40  0001 C CNN "Part Number"
+F 5 "E-Switch" H 12150 4600 40  0001 C CNN "Manufacturer"
+F 6 "SWITCH TACTILE SPST-NO 0.05A 12V" H 12150 4600 40  0001 C CNN "Description"
+F 7 "-20°C +70°C" H 12150 4600 40  0001 C CNN "Temp Range"
+	1    12150 4600
 	1    0    0    -1
 $EndComp
 $Comp
-L JetkovKiCADLib:SM-UART-04L S?
+L JetkovKiCADLib:SM-UART-04L S1
 U 1 1 603C9AA9
 P 12000 5150
-F 0 "S?" H 12078 5188 40  0000 L CNN
+F 0 "S1" H 12078 5188 40  0000 L CNN
 F 1 "SM-UART-04L" H 12078 5112 40  0000 L CNN
 F 2 "JetkovKiCADLib:SM-UART-04L" H 12000 4950 40  0001 C CNN
@@
 	1    0    0    -1
 $EndComp
+$Comp
+L Mechanical:MountingHole H1
+U 1 1 60409DCA
+P 13350 2600
+F 0 "H1" H 13450 2646 50  0000 L CNN
+F 1 "MountingHole" H 13450 2555 50  0000 L CNN
+F 2 "Mounting_Holes:MountingHole_2.2mm_M2" H 13350 2600 50  0001 C CNN
+F 3 "~" H 13350 2600 50  0001 C CNN
+	1    13350 2600
+	1    0    0    -1
+$EndComp

Commit message: Almost final main component placement
Parts:
- removed SW1: TL3301SPF160QJ, JetkovKiCADLib:TL3301EF160QJ, symbol JetkovKiCADLib:TL3301SPF160QG
- added SW1: TL3301SPF160QJ, JetkovKiCADLib:TL3301EF160QJ, symbol JetkovKiCADLib:TL3301SPF160QJ
- D1: footprint JetkovKiCADLib:LED_0603 -> JetkovKiCADLib:155124xx73200; Description LED GREEN CLEAR 0603 SMD -> LED GREEN CLEAR 1204 SMD R/A; Part Number 150060GS75000 -> 155124VS73200; Temp Range (none) -> -40°C +85°C
- D2: value AMBER -> YELLOW; footprint JetkovKiCADLib:LED_0603 -> JetkovKiCADLib:155124xx73200; Description LED AMBER CLEAR 0603 SMD -> LED YELLOW CLEAR 1204 SMD R/A; Part Number 150060AS75000 -> 155124YS73200; Temp Range (none) -> -40°C +85°C
- D3: footprint JetkovKiCADLib:LED_0603 -> JetkovKiCADLib:155124xx73200; Description LED RED CLEAR 0603 SMD -> LED RED CLEAR 1204 SMD R/A; Part Number 150060SS75000 -> 155124RS73200; Temp Range (none) -> -40°C +85°C
Changed lines of the file:
@@
 F 0 "D3" V 5739 6432 50  0000 R CNN
 F 1 "RED" V 5648 6432 50  0000 R CNN
-F 2 "JetkovKiCADLib:LED_0603" H 5700 6550 50  0001 C CNN
-F 3 "https://katalog.we-online.de/led/datasheet/150060SS75000.pdf" H 5700 6550 50  0001 C CNN
-F 4 "150060SS75000" V 5700 6550 50  0001 C CNN "Part Number"
+F 2 "JetkovKiCADLib:155124xx73200" H 5700 6550 50  0001 C CNN
+F 3 "https://katalog.we-online.de/led/datasheet/155124RS73200.pdf" H 5700 6550 50  0001 C CNN
+F 4 "155124RS73200" V 5700 6550 50  0001 C CNN "Part Number"
 F 5 "Wurth Elektronik" V 5700 6550 50  0001 C CNN "Manufacturer"
-F 6 "LED RED CLEAR 0603 SMD" V 5700 6550 50  0001 C CNN "Description"
+F 6 "LED RED CLEAR 1204 SMD R/A" V 5700 6550 50  0001 C CNN "Description"
+F 7 "-40°C +85°C" H 5700 6550 50  0001 C CNN "Temp Range"
 	1    5700 6550
 	0    -1   -1   0
@@
 P 5150 6550
 F 0 "D2" V 5189 6432 50  0000 R CNN
-F 1 "AMBER" V 5098 6432 50  0000 R CNN
-F 2 "JetkovKiCADLib:LED_0603" H 5150 6550 50  0001 C CNN
-F 3 "https://www.we-online.com/catalog/datasheet/150060AS75000.pdf" H 5150 6550 50  0001 C CNN
-F 4 "150060AS75000" V 5150 6550 50  0001 C CNN "Part Number"
+F 1 "YELLOW" V 5098 6432 50  0000 R CNN
+F 2 "JetkovKiCADLib:155124xx73200" H 5150 6550 50  0001 C CNN
+F 3 "https://katalog.we-online.de/led/datasheet/155124YS73200.pdf" H 5150 6550 50  0001 C CNN
+F 4 "155124YS73200" V 5150 6550 50  0001 C CNN "Part Number"
 F 5 "Wurth Elektronik" V 5150 6550 50  0001 C CNN "Manufacturer"
-F 6 "LED AMBER CLEAR 0603 SMD" V 5150 6550 50  0001 C CNN "Description"
+F 6 "LED YELLOW CLEAR 1204 SMD R/A" V 5150 6550 50  0001 C CNN "Description"
+F 7 "-40°C +85°C" H 5150 6550 50  0001 C CNN "Temp Range"
 	1    5150 6550
 	0    -1   -1   0
@@
 F 0 "D1" V 4639 6432 50  0000 R CNN
 F 1 "GREEN" V 4548 6432 50  0000 R CNN
-F 2 "JetkovKiCADLib:LED_0603" H 4600 6550 50  0001 C CNN
-F 3 "https://katalog.we-online.de/led/datasheet/150060GS75000.pdf" H 4600 6550 50  0001 C CNN
-F 4 "150060GS75000" V 4600 6550 50  0001 C CNN "Part Number"
+F 2 "JetkovKiCADLib:155124xx73200" H 4600 6550 50  0001 C CNN
+F 3 "https://katalog.we-online.de/led/datasheet/155124VS73200.pdf" H 4600 6550 50  0001 C CNN
+F 4 "155124VS73200" V 4600 6550 50  0001 C CNN "Part Number"
 F 5 "Wurth Elektronik" V 4600 6550 50  0001 C CNN "Manufacturer"
-F 6 "LED GREEN CLEAR 0603 SMD" V 4600 6550 50  0001 C CNN "Description"
+F 6 "LED GREEN CLEAR 1204 SMD R/A" V 4600 6550 50  0001 C CNN "Description"
+F 7 "-40°C +85°C" H 4600 6550 50  0001 C CNN "Temp Range"
 	1    4600 6550
 	0    -1   -1   0
@@
 $EndComp
 $Comp
-L JetkovKiCADLib:TL3301SPF160QG SW1
-U 1 1 603B5FDC
-P 12150 4600
-F 0 "SW1" H 12150 4885 50  0000 C CNN
-F 1 "TL3301SPF160QJ" H 12150 4794 50  0000 C CNN
-F 2 "JetkovKiCADLib:TL3301EF160QJ" H 12050 4800 50  0001 C CNN
-F 3 "https://www.digikey.ca/htmldatasheets/production/2066007/0/0/1/TL3301SPF160QJ-Drawing.pdf" H 12050 4800 50  0001 C CNN
-F 4 "TL3301SPF160QJ" H 12150 4600 40  0001 C CNN "Part Number"
-F 5 "E-Switch" H 12150 4600 40  0001 C CNN "Manufacturer"
-F 6 "SWITCH TACTILE SPST-NO 0.05A 12V" H 12150 4600 40  0001 C CNN "Description"
-F 7 "-20°C +70°C" H 12150 4600 40  0001 C CNN "Temp Range"
-	1    12150 4600
-	1    0    0    -1
-$EndComp
-$Comp
 L JetkovKiCADLib:SM-UART-04L S1
 U 1 1 603C9AA9
@@
 	1    0    0    -1
 $EndComp
+$Comp
+L JetkovKiCADLib:TL3301SPF160QJ SW1
+U 1 1 604216D1
+P 13100 4600
+F 0 "SW1" H 13100 4885 50  0000 C CNN
+F 1 "TL3301SPF160QJ" H 13100 4794 50  0000 C CNN
+F 2 "JetkovKiCADLib:TL3301EF160QJ" H 13000 4800 50  0001 C CNN
+F 3 "https://www.digikey.ca/htmldatasheets/production/2066007/0/0/1/TL3301SPF160QJ-Drawing.pdf" H 13000 4800 50  0001 C CNN
+F 4 "TL3301SPF160QJ" H 13100 4600 40  0001 C CNN "Part Number"
+F 5 "E-Switch" H 13100 4600 40  0001 C CNN "Manufacturer"
+F 6 "SWITCH TACTILE SPST-NO 0.05A 12V" H 13100 4600 40  0001 C CNN "Description"
+F 7 "-20°C +70°C" H 13100 4600 40  0001 C CNN "Temp Range"
+	1    13100 4600
+	1    0    0    -1
+$EndComp
