File: Canary.sch (KiCad schematic (older format))
At the start: 39 parts, among them J1 CONN_ARM_CM_JTAG_SWD_10, J2 20021311-00010T4LF, Q1 PMN30UNX, Q2 PMN42XPEAH, Q3 PMN30UNX, SW1 TL3301SPF160QJ, U1 BMD-300-A-R, U2 DNP, U3 SHTC3, U4 SGP40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

Commit message: Fill in component info, reduce uniqe resistors. cleanup
Parts:
- R3, R5, R6: value 100k -> 180k; Description RES 100K OHM 1% 1/16W 0402 -> RES 180K OHM 1% 1/16W 0402; Part Number RMCF0402FT100K -> RMCF0402FT180K
- R8, R9: value 100R -> 470R; Description RES 100 OHM 1% 1/16W 0402 -> RES 470 OHM 1% 1/16W 0402; Part Number RMCF0402FT100R -> RMCF0402FT470R
- S1: value SM-UART-04L -> DNP
Changed lines of the file:
@@
 P 1650 6450
 F 0 "R6" H 1720 6496 50  0000 L CNN
-F 1 "100k" H 1720 6405 50  0000 L CNN
+F 1 "180k" H 1720 6405 50  0000 L CNN
 F 2 "JetkovKiCADLib:R_0402_NoSilk" V 1580 6450 50  0001 C CNN
 F 3 "https://www.seielect.com/catalog/sei-rmcf_rmcp.pdf" H 1650 6450 50  0001 C CNN
-F 4 "RES 100K OHM 1% 1/16W 0402" H 1650 6450 50  0001 C CNN "Description"
+F 4 "RES 180K OHM 1% 1/16W 0402" H 1650 6450 50  0001 C CNN "Description"
 F 5 "Stackpole Electronics Inc" H 1650 6450 50  0001 C CNN "Manufacturer"
-F 6 "RMCF0402FT100K" H 1650 6450 50  0001 C CNN "Part Number"
+F 6 "RMCF0402FT180K" H 1650 6450 50  0001 C CNN "Part Number"
 F 7 "-55°C +155°C" H 1650 6450 50  0001 C CNN "Temp Range"
 	1    1650 6450
@@
 P 2150 6450
 F 0 "R8" V 2350 6450 50  0000 L CNN
-F 1 "100R" V 2250 6350 50  0000 L CNN
+F 1 "470R" V 2250 6350 50  0000 L CNN
 F 2 "JetkovKiCADLib:R_0402_NoSilk" V 2080 6450 50  0001 C CNN
 F 3 "https://www.seielect.com/catalog/sei-rmcf_rmcp.pdf" H 2150 6450 50  0001 C CNN
-F 4 "RES 100 OHM 1% 1/16W 0402" H 2150 6450 50  0001 C CNN "Description"
+F 4 "RES 470 OHM 1% 1/16W 0402" H 2150 6450 50  0001 C CNN "Description"
 F 5 "Stackpole Electronics Inc" H 2150 6450 50  0001 C CNN "Manufacturer"
-F 6 "RMCF0402FT100R" H 2150 6450 50  0001 C CNN "Part Number"
+F 6 "RMCF0402FT470R" H 2150 6450 50  0001 C CNN "Part Number"
 F 7 "-55°C +155°C" H 2150 6450 50  0001 C CNN "Temp Range"
 	1    2150 6450
@@
 P 2150 6950
 F 0 "R9" V 2350 6950 50  0000 L CNN
-F 1 "100R" V 2250 6850 50  0000 L CNN
+F 1 "470R" V 2250 6850 50  0000 L CNN
 F 2 "JetkovKiCADLib:R_0402_NoSilk" V 2080 6950 50  0001 C CNN
 F 3 "https://www.seielect.com/catalog/sei-rmcf_rmcp.pdf" H 2150 6950 50  0001 C CNN
-F 4 "RES 100 OHM 1% 1/16W 0402" H 2150 6950 50  0001 C CNN "Description"
+F 4 "RES 470 OHM 1% 1/16W 0402" H 2150 6950 50  0001 C CNN "Description"
 F 5 "Stackpole Electronics Inc" H 2150 6950 50  0001 C CNN "Manufacturer"
-F 6 "RMCF0402FT100R" H 2150 6950 50  0001 C CNN "Part Number"
+F 6 "RMCF0402FT470R" H 2150 6950 50  0001 C CNN "Part Number"
 F 7 "-55°C +155°C" H 2150 6950 50  0001 C CNN "Temp Range"
 	1    2150 6950
@@
 P 8100 3050
 F 0 "S1" H 8178 3088 40  0000 L CNN
-F 1 "SM-UART-04L" H 8178 3012 40  0000 L CNN
+F 1 "DNP" H 8178 3012 40  0000 L CNN
 F 2 "JetkovKiCADLib:SM-UART-04L" H 8100 2850 40  0001 C CNN
 F 3 "https://www.amphenol-sensors.com/en/component/edocman/514-telaire-sm-uart-04l-laser-dust-sensor-application-note/download?Itemid=8488%20%27" H 8100 3050 40  0001 C CNN
@@
 P 1400 5000
 F 0 "R3" H 1470 5046 50  0000 L CNN
-F 1 "100k" H 1470 4955 50  0000 L CNN
+F 1 "180k" H 1470 4955 50  0000 L CNN
 F 2 "JetkovKiCADLib:R_0402_NoSilk" V 1330 5000 50  0001 C CNN
 F 3 "https://www.seielect.com/catalog/sei-rmcf_rmcp.pdf" H 1400 5000 50  0001 C CNN
-F 4 "RES 100K OHM 1% 1/16W 0402" H 1400 5000 50  0001 C CNN "Description"
+F 4 "RES 180K OHM 1% 1/16W 0402" H 1400 5000 50  0001 C CNN "Description"
 F 5 "Stackpole Electronics Inc" H 1400 5000 50  0001 C CNN "Manufacturer"
-F 6 "RMCF0402FT100K" H 1400 5000 50  0001 C CNN "Part Number"
+F 6 "RMCF0402FT180K" H 1400 5000 50  0001 C CNN "Part Number"
 F 7 "-55°C +155°C" H 1400 5000 50  0001 C CNN "Temp Range"
 	1    1400 5000
@@
 AR Path="/60419530" Ref="R5"  Part="1"
 F 0 "R5" V 1777 4736 50  0000 L CNN
-F 1 "100k" V 1700 4700 50  0000 L CNN
+F 1 "180k" V 1700 4700 50  0000 L CNN
 F 2 "JetkovKiCADLib:R_0402_NoSilk" V 1530 4800 50  0001 C CNN
 F 3 "https://www.seielect.com/catalog/sei-rmcf_rmcp.pdf" H 1600 4800 50  0001 C CNN
-F 4 "RES 100K OHM 1% 1/16W 0402" H 1600 4800 50  0001 C CNN "Description"
+F 4 "RES 180K OHM 1% 1/16W 0402" H 1600 4800 50  0001 C CNN "Description"
 F 5 "Stackpole Electronics Inc" H 1600 4800 50  0001 C CNN "Manufacturer"
-F 6 "RMCF0402FT100K" H 1600 4800 50  0001 C CNN "Part Number"
+F 6 "RMCF0402FT180K" H 1600 4800 50  0001 C CNN "Part Number"
 F 7 "-55°C +155°C" H 1600 4800 50  0001 C CNN "Temp Range"
 	1    1600 4800

Commit message: Info tweaks
Other:
- note removed: "TODO\n- Jellybean BOM\n- Review"
Changed lines of the file:
@@
 Wire Wire Line
 	1900 6700 1650 6700
-Text Notes 12100 900  0    118  ~ 0
-TODO\n- Jellybean BOM\n- Review
 Text GLabel 4500 6300 0    50   Input ~ 0
 LED_GREEN

Commit message: Change crystal
Parts:
- Y1: footprint JetkovKiCADLib:FC135327680KAAC3 -> JetkovKiCADLib:FC-12M-327680KA-AC3; Part Number FC-135 32.7680KA-AC3 -> FC-12M 32.7680KA-AC3
Changed lines of the file:
@@
 F 0 "Y1" H 5650 1650 50  0000 C CNN
 F 1 "32.7680 kHz" H 5850 1550 50  0000 C CNN
-F 2 "JetkovKiCADLib:FC135327680KAAC3" H 5350 1550 50  0001 C CNN
-F 3 "https://support.epson.biz/td/api/doc_check.php?dl=brief_FC-135&lang=en" H 5350 1550 50  0001 C CNN
+F 2 "JetkovKiCADLib:FC-12M-327680KA-AC3" H 5350 1550 50  0001 C CNN
+F 3 "https://www.digikey.ca/htmldatasheets/production/1726763/0/0/1/FC-12D-12M-Series-Datasheet.pdf" H 5350 1550 50  0001 C CNN
 F 4 "CRYSTAL 32.7680KHZ 9PF SMD" H 5350 1550 50  0001 C CNN "Description"
 F 5 "EPSON" H 5350 1550 50  0001 C CNN "Manufacturer"
-F 6 "FC-135 32.7680KA-AC3" H 5350 1550 50  0001 C CNN "Part Number"
+F 6 "FC-12M 32.7680KA-AC3" H 5350 1550 50  0001 C CNN "Part Number"
 F 7 "-40°C +85°C" H 5350 1550 50  0001 C CNN "Temp Range"
 	1    5350 1550

Commit message: Change crystal again
Parts:
- Y1: footprint JetkovKiCADLib:FC-12M-327680KA-AC3 -> JetkovKiCADLib:ECS-327-9-12-C-TR; Description CRYSTAL 32.7680KHZ 9PF SMD -> CRYSTAL 32.7680KHZ 9PF 10PPM SMD; Manufacturer EPSON -> ECS Inc.; Part Number FC-12M 32.7680KA-AC3 -> ECS-.327-9-12-C-TR
Changed lines of the file:
@@
 F 0 "Y1" H 5650 1650 50  0000 C CNN
 F 1 "32.7680 kHz" H 5850 1550 50  0000 C CNN
-F 2 "JetkovKiCADLib:FC-12M-327680KA-AC3" H 5350 1550 50  0001 C CNN
-F 3 "https://www.digikey.ca/htmldatasheets/production/1726763/0/0/1/FC-12D-12M-Series-Datasheet.pdf" H 5350 1550 50  0001 C CNN
-F 4 "CRYSTAL 32.7680KHZ 9PF SMD" H 5350 1550 50  0001 C CNN "Description"
-F 5 "EPSON" H 5350 1550 50  0001 C CNN "Manufacturer"
-F 6 "FC-12M 32.7680KA-AC3" H 5350 1550 50  0001 C CNN "Part Number"
+F 2 "JetkovKiCADLib:ECS-327-9-12-C-TR" H 5350 1550 50  0001 C CNN
+F 3 "https://www.ecsxtal.com/store/pdf/ECX_12.pdf" H 5350 1550 50  0001 C CNN
+F 4 "CRYSTAL 32.7680KHZ 9PF 10PPM SMD" H 5350 1550 50  0001 C CNN "Description"
+F 5 "ECS Inc." H 5350 1550 50  0001 C CNN "Manufacturer"
+F 6 "ECS-.327-9-12-C-TR" H 5350 1550 50  0001 C CNN "Part Number"
 F 7 "-40°C +85°C" H 5350 1550 50  0001 C CNN "Temp Range"
 	1    5350 1550

Commit message: Add canary logo
Parts:
- added H2: MountingHole, Mounting_Holes:MountingHole_2.2mm_M2, symbol Mechanical:MountingHole
- added LOGO1: CANARY-LOGO, JetkovKiCADLib:CANARY-LOGO, symbol JetkovKiCADLib:CANARY-LOGO
Changed lines of the file:
@@
 L Mechanical:MountingHole H1
 U 1 1 60409DCA
-P 6550 7050
-F 0 "H1" H 6650 7096 50  0000 L CNN
-F 1 "MountingHole" H 6650 7005 50  0001 L CNN
-F 2 "Mounting_Holes:MountingHole_2.2mm_M2" H 6550 7050 50  0001 C CNN
-F 3 "~" H 6550 7050 50  0001 C CNN
-F 4 "~" H 6550 7050 50  0001 C CNN "Description"
-F 5 "~" H 6550 7050 50  0001 C CNN "Manufacturer"
-F 6 "~" H 6550 7050 50  0001 C CNN "Part Number"
-F 7 "~" H 6550 7050 50  0001 C CNN "Temp Range"
-	1    6550 7050
+P 6550 6800
+F 0 "H1" H 6650 6846 50  0000 L CNN
+F 1 "MountingHole" H 6650 6755 50  0001 L CNN
+F 2 "Mounting_Holes:MountingHole_2.2mm_M2" H 6550 6800 50  0001 C CNN
+F 3 "~" H 6550 6800 50  0001 C CNN
+F 4 "~" H 6550 6800 50  0001 C CNN "Description"
+F 5 "~" H 6550 6800 50  0001 C CNN "Manufacturer"
+F 6 "~" H 6550 6800 50  0001 C CNN "Part Number"
+F 7 "~" H 6550 6800 50  0001 C CNN "Temp Range"
+	1    6550 6800
 	1    0    0    -1
 $EndComp
@@
 	1    0    0    -1
 $EndComp
+$Comp
+L Mechanical:MountingHole H2
+U 1 1 60576303
+P 6550 7050
+F 0 "H2" H 6650 7096 50  0000 L CNN
+F 1 "MountingHole" H 6650 7005 50  0001 L CNN
+F 2 "Mounting_Holes:MountingHole_2.2mm_M2" H 6550 7050 50  0001 C CNN
+F 3 "~" H 6550 7050 50  0001 C CNN
+F 4 "~" H 6550 7050 50  0001 C CNN "Description"
+F 5 "~" H 6550 7050 50  0001 C CNN "Manufacturer"
+F 6 "~" H 6550 7050 50  0001 C CNN "Part Number"
+F 7 "~" H 6550 7050 50  0001 C CNN "Temp Range"
+	1    6550 7050
+	1    0    0    -1
+$EndComp
+$Comp
+L JetkovKiCADLib:CANARY-LOGO LOGO1
+U 1 1 60599864
+P 6550 7300
+F 0 "LOGO1" H 6628 7300 40  0000 L CNN
+F 1 "CANARY-LOGO" H 6550 7200 40  0001 C CNN
+F 2 "JetkovKiCADLib:CANARY-LOGO" H 6550 7100 40  0001 C CNN
+F 3 "" H 6550 7300 40  0001 C CNN
+	1    6550 7300
+	1    0    0    -1
+$EndComp

Commit message: Add TVS diodes, resistor for piezo drive, and test point
Parts:
- added D5, D6: D_Schottky_ALT, JetkovKiCADLib:NSPU3051, symbol Device:D_Schottky_ALT
- added R30: 487k, JetkovKiCADLib:R_0402_NoSilk, symbol Device:R
- added TP1: TestPoint, Measurement_Points:Measurement_Point_Round-SMD-Pad_Small, symbol Connector:TestPoint
Connections:
- wire segments 132 -> 137
- no-connect marks 9 -> 8
Other:
- note added: "Assume 20pF capacitance\n4kHz -> 250us = 20T\n250us / 20 = RC -> R = 625k"
Changed lines of the file:
@@
 	1900 6700 1900 6950
-Wire Wire Line
-	2600 6650 2600 6700
 Wire Wire Line
 	1650 6600 1650 6700
@@
 Wire Wire Line
 	2600 7150 2600 7200
-Wire Wire Line
-	3000 6700 2600 6700
-Connection ~ 2600 6700
-Wire Wire Line
-	2600 6700 2600 6750
-Wire Wire Line
-	3000 6800 2950 6800
-Wire Wire Line
-	2950 6800 2950 7200
-$Comp
-L power:GND #PWR018
-U 1 1 6069713F
-P 2950 7200
-F 0 "#PWR018" H 2950 6950 50  0001 C CNN
-F 1 "GND" H 2955 7027 50  0000 C CNN
-F 2 "" H 2950 7200 50  0001 C CNN
-F 3 "" H 2950 7200 50  0001 C CNN
-	1    2950 7200
-	1    0    0    -1
-$EndComp
 Wire Wire Line
 	2000 6450 1900 6450
@@
 U 1 1 603AA039
 P 2500 6450
-F 0 "Q2" H 2705 6450 50  0000 L CNN
+F 0 "Q2" H 2450 6250 50  0000 L CNN
 F 1 "PMN42XPEAH" H 2705 6405 50  0001 L CNN
 F 2 "JetkovKiCADLib:PMN-NXP-TSOP6-SOT457" H 2600 5800 50  0001 C CNN
@@
 U 1 1 603AB800
 P 2500 6950
-F 0 "Q3" H 2705 6950 50  0000 L CNN
+F 0 "Q3" H 2450 6750 50  0000 L CNN
 F 1 "PMN30UNX" H 2705 6905 50  0001 L CNN
 F 2 "JetkovKiCADLib:PMN-NXP-TSOP6-SOT457" H 2650 6350 50  0001 C CNN
@@
 Text Notes 750  5850 0    79   Italic 0
 Indication
-Text Notes 3400 6850 0    79   ~ 0
-Pizeo\nBuzzer
 $Comp
 L Device:C C8
@@
 Text GLabel 5550 4850 2    50   Input ~ 0
 SPI_MOSI
-Text GLabel 5550 4950 2    50   Input ~ 0
+Text GLabel 5550 4950 2    50   Output ~ 0
 SPI_MISO
 Text GLabel 5550 4750 2    50   Input ~ 0
@@
 Text GLabel 7350 3450 0    50   Input ~ 0
 PM_UART_RXD
-Text GLabel 7350 3550 0    50   Input ~ 0
+Text GLabel 7350 3550 0    50   Output ~ 0
 PM_UART_TXD
 $Comp
@@
 	1    0    0    -1
 $EndComp
-Text GLabel 2700 2550 0    50   Input ~ 0
+Text GLabel 2700 2550 0    50   Output ~ 0
 PM_UART_RXD
 Text GLabel 2700 2650 0    50   Input ~ 0
@@
 Text GLabel 7950 3500 2    35   Input ~ 0
 ~PM_SLEEP~
-Text GLabel 2700 2750 0    35   Input ~ 0
+Text GLabel 2700 2750 0    35   Output ~ 0
 ~PM_SLEEP~
 Text GLabel 1250 2950 0    50   Input ~ 0
@@
 Wire Wire Line
 	1500 2950 1250 2950
-Text GLabel 2700 2350 0    50   Input ~ 0
+Text GLabel 2700 2350 0    50   Output ~ 0
 LED_AMBER
-Text GLabel 2700 2250 0    50   Input ~ 0
+Text GLabel 2700 2250 0    50   Output ~ 0
 LED_RED
-Text GLabel 2700 2450 0    50   Input ~ 0
+Text GLabel 2700 2450 0    50   Output ~ 0
 LED_GREEN
 Text GLabel 4500 3050 2    50   Input ~ 0
@@
 Text GLabel 2700 3450 0    35   Input ~ 0
 ~FLASH_CS~
-Text GLabel 2700 3250 0    50   Input ~ 0
+Text GLabel 2700 3250 0    50   Output ~ 0
 SPI_MOSI
 Text GLabel 2700 3350 0    50   Input ~ 0
 SPI_MISO
-Text GLabel 2700 3150 0    50   Input ~ 0
+Text GLabel 2700 3150 0    50   Output ~ 0
 SPI_CLK
 Text GLabel 4500 2650 2    35   Output ~ 0
@@
 Text Label 4500 1350 0    40   ~ 0
 XTAL1
-Text Label 2700 6700 0    40   ~ 0
-PDRIVE_O
 Text Label 1650 6700 0    40   ~ 0
 PDRIVE
-$Comp
-L JetkovKiCADLib:PKMCS0909E4000-R1 LS1
-U 1 1 603826A5
-P 3200 6700
-F 0 "LS1" H 3100 6850 50  0000 L CNN
-F 1 "PKMCS0909E4000-R1" H 3100 6350 50  0000 L CNN
-F 2 "JetkovKiCADLib:PKMCS0909E4000-R1" H 3215 6350 50  0001 C CNN
-F 3 "https://www.murata.com/~/media/webrenewal/products/sound/sounder/vppt-buzj083-d.ashx" H 3165 6650 50  0001 C CNN
-F 4 "PKMCS0909E4000-R1" H 3150 6400 40  0001 C CNN "Part Number"
-F 5 "Murata Electronics" H 3150 6400 40  0001 C CNN "Manufacturer"
-F 6 "AUDIO PIEZO TRANSDUCER 12.5V SMD" H 3250 6400 40  0001 C CNN "Description"
-F 7 "-40°C +85°C" H 3150 6400 40  0001 C CNN "Temp Range"
-	1    3200 6700
-	1    0    0    -1
-$EndComp
 $Comp
 L JetkovKiCADLib:20021311-00010T4LF J2
@@
 Button
 NoConn ~ 2700 1750
-NoConn ~ 2700 1850
 Wire Wire Line
 	2750 1750 2700 1750
@@
 	1    0    0    -1
 $EndComp
+$Comp
+L Connector:TestPoint TP1
+U 1 1 603E3FCA
+P 2700 1850
+F 0 "TP1" V 2781 1905 50  0000 L CNN
+F 1 "TestPoint" H 2758 1877 50  0001 L CNN
+F 2 "Measurement_Points:Measurement_Point_Round-SMD-Pad_Small" H 2900 1850 50  0001 C CNN
+F 3 "~" H 2900 1850 50  0001 C CNN
+	1    2700 1850
+	0    -1   -1   0
+$EndComp
+Text Notes 2900 7750 0    40   ~ 0
+Assume 20pF capacitance\n4kHz -> 250us = 20T\n250us / 20 = RC -> R = 625k
+$Comp
+L JetkovKiCADLib:PKMCS0909E4000-R1 LS1
+U 1 1 603826A5
+P 3550 6700
+F 0 "LS1" H 3450 6850 50  0000 L CNN
+F 1 "PKMCS0909E4000-R1" H 3450 6350 50  0000 L CNN
+F 2 "JetkovKiCADLib:PKMCS0909E4000-R1" H 3565 6350 50  0001 C CNN
+F 3 "https://www.murata.com/~/media/webrenewal/products/sound/sounder/vppt-buzj083-d.ashx" H 3515 6650 50  0001 C CNN
+F 4 "PKMCS0909E4000-R1" H 3500 6400 40  0001 C CNN "Part Number"
+F 5 "Murata Electronics" H 3500 6400 40  0001 C CNN "Manufacturer"
+F 6 "AUDIO PIEZO TRANSDUCER 12.5V SMD" H 3600 6400 40  0001 C CNN "Description"
+F 7 "-40°C +85°C" H 3500 6400 40  0001 C CNN "Temp Range"
+	1    3550 6700
+	1    0    0    -1
+$EndComp
+Text Notes 3750 6850 0    79   ~ 0
+Pizeo\nBuzzer
+$Comp
+L power:GND #PWR018
+U 1 1 6069713F
+P 3300 7200
+F 0 "#PWR018" H 3300 6950 50  0001 C CNN
+F 1 "GND" H 3305 7027 50  0000 C CNN
+F 2 "" H 3300 7200 50  0001 C CNN
+F 3 "" H 3300 7200 50  0001 C CNN
+	1    3300 7200
+	1    0    0    -1
+$EndComp
+Wire Wire Line
+	3300 6800 3300 7200
+Wire Wire Line
+	3350 6800 3300 6800
+Wire Wire Line
+	2600 6650 2600 6700
+$Comp
+L Device:R R?
+U 1 1 603FF1FC
+P 2900 6700
+AR Path="/60656A7D/603FF1FC" Ref="R?"  Part="1"
+AR Path="/603FF1FC" Ref="R30"  Part="1"
+F 0 "R30" V 3070 6683 50  0000 L CNN
+F 1 "487k" V 2986 6610 50  0000 L CNN
+F 2 "JetkovKiCADLib:R_0402_NoSilk" V 2830 6700 50  0001 C CNN
+F 3 "https://www.seielect.com/catalog/sei-rmcf_rmcp.pdf" H 2900 6700 50  0001 C CNN
+F 4 "RES 487K OHM 1% 1/16W 0402" H 2900 6700 50  0001 C CNN "Description"
+F 5 "Stackpole Electronics Inc" H 2900 6700 50  0001 C CNN "Manufacturer"
+F 6 "RMCF0402FT487K" H 2900 6700 50  0001 C CNN "Part Number"
+F 7 "-55°C +155°C" H 2900 6700 50  0001 C CNN "Temp Range"
+	1    2900 6700
+	0    -1   -1   0
+$EndComp
+Text Label 3100 6700 0    40   ~ 0
+PDRIVE_O
+$Comp
+L Device:D_Schottky_ALT D6
+U 1 1 603EE231
+P 3100 6950
+F 0 "D6" V 3100 7075 50  0000 C CNN
+F 1 "D_Schottky_ALT" H 3100 7076 50  0001 C CNN
+F 2 "JetkovKiCADLib:NSPU3051" H 3100 6950 50  0001 C CNN
+F 3 "http://www.onsemi.com/pub/Collateral/NSPU3051-D.PDF" H 3100 6950 50  0001 C CNN
+F 4 "TVS DIODE 5.5V 9.5V 2X2DFN" H 3100 6950 50  0001 C CNN "Description"
+F 5 "ON Semiconductor" H 3100 6950 50  0001 C CNN "Manufacturer"
+F 6 "NSPU3051N2T5G" H 3100 6950 50  0001 C CNN "Part Number"
+F 7 "-65°C +150°C" H 3100 6950 50  0001 C CNN "Temp Range"
+	1    3100 6950
+	0    -1   1    0
+$EndComp
+Connection ~ 2600 6700
+Wire Wire Line
+	2600 6700 2600 6750
+Wire Wire Line
+	2600 6700 2750 6700
+Wire Wire Line
+	3350 6700 3100 6700
+Wire Wire Line
+	3100 6700 3100 6800
+Connection ~ 3100 6700
+Wire Wire Line
+	3100 6700 3050 6700
+$Comp
+L power:GND #PWR084
+U 1 1 60457D08
+P 3100 7200
+F 0 "#PWR084" H 3100 6950 50  0001 C CNN
+F 1 "GND" H 3105 7027 50  0000 C CNN
+F 2 "" H 3100 7200 50  0001 C CNN
+F 3 "" H 3100 7200 50  0001 C CNN
+	1    3100 7200
+	1    0    0    -1
+$EndComp
+Wire Wire Line
+	3100 7200 3100 7100
+$Comp
+L Device:D_Schottky_ALT D5
+U 1 1 60463B42
+P 1200 5000
+F 0 "D5" V 1200 5125 50  0000 C CNN
+F 1 "D_Schottky_ALT" H 1200 5126 50  0001 C CNN
+F 2 "JetkovKiCADLib:NSPU3051" H 1200 5000 50  0001 C CNN
+F 3 "http://www.onsemi.com/pub/Collateral/NSPU3051-D.PDF" H 1200 5000 50  0001 C CNN
+F 4 "TVS DIODE 5.5V 9.5V 2X2DFN" H 1200 5000 50  0001 C CNN "Description"
+F 5 "ON Semiconductor" H 1200 5000 50  0001 C CNN "Manufacturer"
+F 6 "NSPU3051N2T5G" H 1200 5000 50  0001 C CNN "Part Number"
+F 7 "-65°C +150°C" H 1200 5000 50  0001 C CNN "Temp Range"
+	1    1200 5000
+	0    -1   1    0
+$EndComp
+Wire Wire Line
+	1200 4850 1200 4800
+Connection ~ 1200 4800
+$Comp
+L power:GND #PWR083
+U 1 1 6046F176
+P 1200 5150
+F 0 "#PWR083" H 1200 4900 50  0001 C CNN
+F 1 "GND" H 1205 4977 50  0000 C CNN
+F 2 "" H 1200 5150 50  0001 C CNN
+F 3 "" H 1200 5150 50  0001 C CNN
+	1    1200 5150
+	1    0    0    -1
+$EndComp

Commit message: Clean up silks, add fiducials
Parts:
- added FID1, FID2, FID3, FID4, FID5, FID6: Fiducial, Fiducials:Fiducial_1mm_Dia_2mm_Outer, symbol Mechanical:Fiducial
Changed lines of the file:
@@
 L Mechanical:MountingHole H1
 U 1 1 60409DCA
-P 6550 6800
-F 0 "H1" H 6650 6846 50  0000 L CNN
-F 1 "MountingHole" H 6650 6755 50  0001 L CNN
-F 2 "Mounting_Holes:MountingHole_2.2mm_M2" H 6550 6800 50  0001 C CNN
-F 3 "~" H 6550 6800 50  0001 C CNN
-F 4 "~" H 6550 6800 50  0001 C CNN "Description"
-F 5 "~" H 6550 6800 50  0001 C CNN "Manufacturer"
-F 6 "~" H 6550 6800 50  0001 C CNN "Part Number"
-F 7 "~" H 6550 6800 50  0001 C CNN "Temp Range"
-	1    6550 6800
+P 6300 6600
+F 0 "H1" H 6400 6600 50  0000 L CNN
+F 1 "MountingHole" H 6400 6555 50  0001 L CNN
+F 2 "Mounting_Holes:MountingHole_2.2mm_M2" H 6300 6600 50  0001 C CNN
+F 3 "~" H 6300 6600 50  0001 C CNN
+F 4 "~" H 6300 6600 50  0001 C CNN "Description"
+F 5 "~" H 6300 6600 50  0001 C CNN "Manufacturer"
+F 6 "~" H 6300 6600 50  0001 C CNN "Part Number"
+F 7 "~" H 6300 6600 50  0001 C CNN "Temp Range"
+	1    6300 6600
 	1    0    0    -1
 $EndComp
@@
 L Mechanical:MountingHole H2
 U 1 1 60576303
-P 6550 7050
-F 0 "H2" H 6650 7096 50  0000 L CNN
-F 1 "MountingHole" H 6650 7005 50  0001 L CNN
-F 2 "Mounting_Holes:MountingHole_2.2mm_M2" H 6550 7050 50  0001 C CNN
-F 3 "~" H 6550 7050 50  0001 C CNN
-F 4 "~" H 6550 7050 50  0001 C CNN "Description"
-F 5 "~" H 6550 7050 50  0001 C CNN "Manufacturer"
-F 6 "~" H 6550 7050 50  0001 C CNN "Part Number"
-F 7 "~" H 6550 7050 50  0001 C CNN "Temp Range"
-	1    6550 7050
+P 6650 6600
+F 0 "H2" H 6750 6600 50  0000 L CNN
+F 1 "MountingHole" H 6750 6555 50  0001 L CNN
+F 2 "Mounting_Holes:MountingHole_2.2mm_M2" H 6650 6600 50  0001 C CNN
+F 3 "~" H 6650 6600 50  0001 C CNN
+F 4 "~" H 6650 6600 50  0001 C CNN "Description"
+F 5 "~" H 6650 6600 50  0001 C CNN "Manufacturer"
+F 6 "~" H 6650 6600 50  0001 C CNN "Part Number"
+F 7 "~" H 6650 6600 50  0001 C CNN "Temp Range"
+	1    6650 6600
 	1    0    0    -1
 $EndComp
@@
 L JetkovKiCADLib:CANARY-LOGO LOGO1
 U 1 1 60599864
-P 6550 7300
-F 0 "LOGO1" H 6628 7300 40  0000 L CNN
-F 1 "CANARY-LOGO" H 6550 7200 40  0001 C CNN
-F 2 "JetkovKiCADLib:CANARY-LOGO" H 6550 7100 40  0001 C CNN
-F 3 "" H 6550 7300 40  0001 C CNN
-	1    6550 7300
+P 6500 6800
+F 0 "LOGO1" H 6578 6800 40  0000 L CNN
+F 1 "CANARY-LOGO" H 6500 6700 40  0001 C CNN
+F 2 "JetkovKiCADLib:CANARY-LOGO" H 6500 6600 40  0001 C CNN
+F 3 "" H 6500 6800 40  0001 C CNN
+	1    6500 6800
 	1    0    0    -1
 $EndComp
@@
 	1    0    0    -1
 $EndComp
+$Comp
+L Mechanical:Fiducial FID1
+U 1 1 60420BD8
+P 6300 7000
+F 0 "FID1" H 6385 7000 50  0000 L CNN
+F 1 "Fiducial" H 6385 6955 50  0001 L CNN
+F 2 "Fiducials:Fiducial_1mm_Dia_2mm_Outer" H 6300 7000 50  0001 C CNN
+F 3 "~" H 6300 7000 50  0001 C CNN
+	1    6300 7000
+	1    0    0    -1
+$EndComp
+$Comp
+L Mechanical:Fiducial FID2
+U 1 1 60421C0D
+P 6300 7150
+F 0 "FID2" H 6385 7150 50  0000 L CNN
+F 1 "Fiducial" H 6385 7105 50  0001 L CNN
+F 2 "Fiducials:Fiducial_1mm_Dia_2mm_Outer" H 6300 7150 50  0001 C CNN
+F 3 "~" H 6300 7150 50  0001 C CNN
+	1    6300 7150
+	1    0    0    -1
+$EndComp
+$Comp
+L Mechanical:Fiducial FID3
+U 1 1 604274F6
+P 6300 7300
+F 0 "FID3" H 6385 7300 50  0000 L CNN
+F 1 "Fiducial" H 6385 7255 50  0001 L CNN
+F 2 "Fiducials:Fiducial_1mm_Dia_2mm_Outer" H 6300 7300 50  0001 C CNN
+F 3 "~" H 6300 7300 50  0001 C CNN
+	1    6300 7300
+	1    0    0    -1
+$EndComp
+$Comp
+L Mechanical:Fiducial FID4
+U 1 1 6042CD9B
+P 6650 7000
+F 0 "FID4" H 6735 7000 50  0000 L CNN
+F 1 "Fiducial" H 6735 6955 50  0001 L CNN
+F 2 "Fiducials:Fiducial_1mm_Dia_2mm_Outer" H 6650 7000 50  0001 C CNN
+F 3 "~" H 6650 7000 50  0001 C CNN
+	1    6650 7000
+	1    0    0    -1
+$EndComp
+$Comp
+L Mechanical:Fiducial FID5
+U 1 1 604325C6
+P 6650 7150
+F 0 "FID5" H 6735 7150 50  0000 L CNN
+F 1 "Fiducial" H 6735 7105 50  0001 L CNN
+F 2 "Fiducials:Fiducial_1mm_Dia_2mm_Outer" H 6650 7150 50  0001 C CNN
+F 3 "~" H 6650 7150 50  0001 C CNN
+	1    6650 7150
+	1    0    0    -1
+$EndComp
+$Comp
+L Mechanical:Fiducial FID6
+U 1 1 60437D6F
+P 6650 7300
+F 0 "FID6" H 6735 7300 50  0000 L CNN
+F 1 "Fiducial" H 6735 7255 50  0001 L CNN
+F 2 "Fiducials:Fiducial_1mm_Dia_2mm_Outer" H 6650 7300 50  0001 C CNN
+F 3 "~" H 6650 7300 50  0001 C CNN
+	1    6650 7300
+	1    0    0    -1
+$EndComp
